File: currentdumping2.kicad_sch (KiCad schematic)
At the start: 18 parts, among them J101 POWER, J102 LEFT_IN, J103 RIGHT_IN, J104 LEFT_OUT, J105 RIGHT_OUT, Q101 2N5551, Q102 2N5401, U101 OPA2134

Commit message: Fill attributes in schematic
Other:
- company: (none) -> jxdking
- title: (none) -> 2nd Order Current Dumping
Changed lines of the file:
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@@
 	(generator "eeschema")
 	(generator_version "10.0")
-	(paper "A4")
+	(paper "USLetter")
+	(title_block
+		(title "2nd Order Current Dumping")
+		(rev "202610A")
+		(company "jxdking")
+	)
 	(junction
 		(at 140.97 58.42)
