File: currentdumping2.kicad_pcb (KiCad board)
At the start: 2 copper layers, 140 x 100 mm, 118 parts, among them J101 POWER, J102 LEFT_IN, J103 RIGHT_IN, J104 LEFT_OUT, J105 RIGHT_OUT, Q101 2N5551, Q102 2N5401, Q201 2N5551, Q202 2N5401, Q203 2N5551, Q204 2N5551, Q205 2N5401, Q206 2N5401, Q207 2N5401, Q208 2N5551, Q209 MJE340, Q210 MJE340, Q211 MJE350, Q212 MJW3281, Q213 MJW1302, Q301 2N5551, Q302 2N5401, Q303 2N5551, Q304 2N5551, Q305 2N5401, Q306 2N5401, Q307 2N5401, Q308 2N5551, Q309 MJE340, Q310 MJE340, Q311 MJE350, Q312 MJW3281, Q313 MJW1302, U101 OPA2134

Commit message: Add polarity labels to the connector footprints
Other:
- board text added: "+"
- board text added: "-"
- board text added: "GND"
- board text added: "SGND"
